File: hardware/custom-wireless-mouse.kicad_sch (KiCad schematic)
At the start: 33 parts, among them J1 SWD_HEADER, J2 B2B-XH-A, Q1 DMP2035U, SW1 JS202011SCQN, SW2 EVQ-P7B01P, SW3 EVQ-P7B01P, SW4 EVQ-P7B01P, U1 nRF52810-QCAA-T, U2 PMW3610DM-SUDU, U3 TLV61220DBVT, Y1 NX2016SA-32MHZ

Commit message: Replace SW2-4/ENC1 with DIY-compatible switch and real scroll encoder
Researched against real datasheets and the DIY mouse-modding market:
Panasonic EVQ-P7B01P (SW2-4) is an SMD tactile switch in a fundamentally
different, much smaller footprint than any common 2-pin/3-pin mouse
micro switch (Omron D2FC, Kailh GM series, Huano, TTC all share one
~12.8x5.8x6.5mm through-hole body) - no swap-in flexibility was actually
possible with it. Bourns PEC11R-4220F-S0012 (ENC1) is vertical-mount
only with an oversized 6mm shaft - wrong orientation and wrong diameter
for a flat-PCB mouse scroll wheel, though its built-in pushbutton did
work.

Replaced with:
- SW2-4 (L/R/FN) and new SW5 (wheel middle-click): Omron D2FC-F-7N(20M),
  hand-drawn footprint from Omron's own published D2F-family mechanical
  drawing - the shared body the whole DIY mouse-switch aftermarket
  clones, so 2-pin or 3-pin swap-in switches solder on directly.
- ENC1: a TTC/Kailh-style mouse scroll wheel encoder with the correct
  ~1.74mm shaft for a real wheel hub. No official datasheet exists for
  this part class (mod-market only) - its footprint is an explicit,
  clearly-documented placeholder pending physical measurement, same
  treatment as L1's existing placeholder footprint. No built-in
  pushbutton, hence SW5.

All five new parts are placed on the schematic but deliberately left
unwired. Docs (bom.md, pinout.md, schematic.md, open-items.md,
kicad-build-guide.md) updated throughout to match.
Parts:
- removed ENC1: PEC11R-4220F-S0012, bourns-pec11r:rotary-encoder-switched-pec11r, symbol bourns-pec11r:PEC11R-4220F-S0012
- removed SW2, SW3, SW4: EVQ-P7B01P, panasonic-evq-p7b01p:sw-spst-evqp7-side-actuated, symbol panasonic-evq-p7b01p:EVQ-P7B01P
- added ENC1: MOUSE_ENCODER, ttc-kailh-mouse-encoder:encoder-tht-placeholder-mouse-wheel, symbol ttc-kailh-mouse-encoder:MOUSE_ENCODER
- added SW2, SW3, SW4, SW5: D2FC-F-7N(20M), omron-d2fc-f-7n:switch-tht-omron-d2fc-f-7n, symbol omron-d2fc-f-7n:D2FC-F-7N-20M
- C12, C8: value 10uF X7R -> 10uF
- C13: value 10nF X7R -> 10nF
- R1: value 10k DNI -> 10k
Other:
- note removed: "DCC: unconnected (LDO only)"
- note removed: "LENS1 (PixArt LM18-LSI) — mechanical only, no schematic connection"
- note removed: "PCB trace antenna (see docs/hardware/architecture.md)"
- note removed: "R1: optional / DNI — PMW3610 has an internal weak pull-up on NRESET"
- note removed: "VOUT (R2/R3 divider) targets ~1.9V (margin above TLV61220's 1.8V floor) see docs/hardware/bom.md"
- moved on the sheet: C1, C10, C11, C12, C13, C14, C2, C3, C4, C5, C8, C9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
