File: hardware/custom-wireless-mouse.kicad_sch (KiCad schematic)
At the start: 34 parts, among them J1 SWD_HEADER, J2 B2B-XH-A, Q1 DMG2305UXQ, SW1 JS202011SCQN, SW2 D2FC-F-7N(20M), SW3 D2FC-F-7N(20M), SW4 D2FC-F-7N(20M), SW5 B3U-1000P, U1 nRF52810-QCAA-T, U2 PMW3610DM-SUDU, U3 TLV61220DBVT, Y1 NX2016SA-32MHZ

Commit message: First-pass routing, remove function button, rewire SW5
Routed the board (ENC1/SW2/SW3/SW5/U1/U3/J1/J2/Q1/antenna feed all
connected) and placed a meandered PCB trace antenna. DRC dropped from
13 violations / 53 unconnected items to 1 violation / 0 unconnected.

Removed SW4 (function/DPI button) for lack of routing space -- dropped
its footprint, its BTN_FN net, and the now-stale references across
docs. U1 pin 15 (P0.20) is now a spare no-connect GPIO. Any DPI/secondary
function will need to be remapped onto the remaining buttons in firmware.

Rewired SW5 (pin 1 -> BTN_SCRL, pin 2 -> GND, matching the old D2FC's
mapping) and placed it on the PCB next to ENC1.

Logged the one remaining DRC error in open-items.md: the antenna feed
trace clips the board's own "Antenna" keepout zone, which currently
disallows tracks/vias there as well as copper pour -- needs a layout
decision, not a doc fix.

Co-Authored-By: Claude Sonnet 5 <noreply@anthropic.com>
Parts:
- removed SW4: D2FC-F-7N(20M), omron-d2fc-f-7n:switch-tht-omron-d2fc-f-7n, symbol omron-d2fc-f-7n:D2FC-F-7N-20M
Connections:
- net BTN_FN: no longer names the net of U1.15 (P0.20)
